File: psu.kicad_sch (KiCad schematic)
At the start: 42 parts, among them U401 XL1509, U402 XL1509

Commit message: finish layout
Parts:
- added C? (x6): 10uF, Capacitor_SMD:C_0603_1608Metric, symbol Device:C_Small
- C414, C415, C420, C421, C? (x2): footprint (none) -> Capacitor_SMD:CP_Elec_8x10.5
- C416, C417, C418, C419, C? (x11): footprint (none) -> Capacitor_SMD:C_0603_1608Metric
- D401, D402, D404: footprint (none) -> Diode_SMD:D_0603_1608Metric
- D403, D405, D406: footprint (none) -> Diode_SMD:D_SMA
- J?: footprint (none) -> easyeda2kicad:DC-IN-TH_DC-005-5A-2.0-SMT
- L401, L402: footprint (none) -> Inductor_SMD:L_12x12mm_H8mm
- R401, R402, R403, R404, R405, R406: footprint (none) -> Resistor_SMD:R_0603_1608Metric
- R407: value 1.69k -> 1.8k; footprint (none) -> Resistor_SMD:R_0603_1608Metric
- TP401, TP402, TP403: footprint (none) -> TestPoint:TestPoint_Pad_D1.0mm
- U401, U402: footprint (none) -> Package_SO:SOIC-8_3.9x4.9mm_P1.27mm
Connections:
- net +12V: now also C?.1, C?.1, C?.1, C?.1, C?.1, C?.1
- net GND: now also C?.2, C?.2, C?.2, C?.2, C?.2, C?.2
Other:
- moved on the sheet: C?, D403, J?, TP402
