File: alignment.kicad_sch (KiCad schematic)
At the start: 19 parts, among them J202 P3, J203 P2, J205 P6

Commit message: finish layout
Parts:
- added JP?: EOL_VCC, Jumper:SolderJumper-3_P1.3mm_Bridged12_RoundedPad1.0x1.5mm, symbol Jumper:SolderJumper_3_Bridged12
- added TP301: EOL_LEFT, TestPoint:TestPoint_Pad_D1.0mm, symbol Connector:TestPoint
- added TP302: EOL_RIGHT, TestPoint:TestPoint_Pad_D1.0mm, symbol Connector:TestPoint
- C301, C302: footprint (none) -> Capacitor_SMD:C_0603_1608Metric
- D301, D302: footprint (none) -> Diode_SMD:D_MiniMELF
- J202: footprint (none) -> Connector_JST:JST_XH_B5B-XH-A_1x05_P2.50mm_Vertical
- J203, J205: footprint (none) -> Connector_JST:JST_XH_B3B-XH-A_1x03_P2.50mm_Vertical
- JP? (x3): footprint (none) -> Jumper:SolderJumper-3_P1.3mm_Bridged12_RoundedPad1.0x1.5mm
- R307, R308: value 665R -> 680R; footprint (none) -> Resistor_SMD:R_0603_1608Metric
- R? (x6): footprint (none) -> Resistor_SMD:R_0603_1608Metric
Connections:
- net +3V3: now also JP?.3 (B)
- net +5V: now also JP?.1 (A)
- net BELT_PHASE: now also U?.10 (A8); no longer U?.5 (A3)
- net ENC_B: now also U?.18 (B4); no longer U?.20 (B2)
- net ENC_BP: now also U?.14 (B8); no longer U?.19 (B3)
- net ENC_V1: now also U?.6 (A4); no longer U?.4 (A2)
- net EOL_LEFT: now also TP301.1
- net EOL_RIGHT: now also TP302.1
- net GND: now also U?.4 (A2), U?.5 (A3); no longer U?.10 (A8), U?.6 (A4)
- net at J203.2 (Pin_2), JP?.2 (C): no longer J205.2 (Pin_2)
- new net: J205.2 (Pin_2), JP?.2 (C)
- no-connect marks 0 -> 5
Other:
- moved on the sheet: JP?, R?

Commit message: finalize fab files and order first rev of board
Parts:
- J202, J203, J205: now left out of the parts list
Changed lines of the file:
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@@
   )
   (symbol (lib_id "Connector_Generic:Conn_01x03") (at 172.72 49.53 0) (unit 1)
-    (in_bom yes) (on_board yes) (dnp no) (fields_autoplaced)
+    (in_bom no) (on_board yes) (dnp no) (fields_autoplaced)
     (property "Reference" "J205" (at 175.26 48.895 0)
       (effects (font (size 1.27 1.27)) (justify left))
@@
   )
   (symbol (lib_id "Connector_Generic:Conn_01x05") (at 172.72 72.39 0) (unit 1)
-    (in_bom yes) (on_board yes) (dnp no) (fields_autoplaced)
+    (in_bom no) (on_board yes) (dnp no) (fields_autoplaced)
     (property "Reference" "J202" (at 175.26 71.755 0)
       (effects (font (size 1.27 1.27)) (justify left))
@@
   )
   (symbol (lib_id "Connector_Generic:Conn_01x03") (at 172.72 31.75 0) (unit 1)
-    (in_bom yes) (on_board yes) (dnp no) (fields_autoplaced)
+    (in_bom no) (on_board yes) (dnp no) (fields_autoplaced)
     (property "Reference" "J203" (at 175.26 31.115 0)
       (effects (font (size 1.27 1.27)) (justify left))
