File: solenoids.kicad_sch (KiCad schematic)
At the start: 86 parts, among them J201 P4, J202 P5

Commit message: finish layout
Parts:
- removed TP201, TP204, TP205, TP206, TP207, TP210, TP211, TP212, TP213, TP214, TP215, TP216, TP217, TP218, TP219, TP220, TP221, TP222, TP223, TP224: AUX0, symbol Connector:TestPoint
- removed TP202, TP208: AUX1, symbol Connector:TestPoint
- removed TP203, TP209: AUX2, symbol Connector:TestPoint
- J?: renamed from J201; footprint (none) -> Connector_JST:JST_XH_B8B-XH-A_1x08_P2.50mm_Vertical
- J?: renamed from J202; footprint (none) -> Connector_JST:JST_XH_B10B-XH-A_1x10_P2.50mm_Vertical
- R? (x56): footprint (none) -> Resistor_SMD:R_0603_1608Metric
- U? (x4): footprint (none) -> Package_SO:SOIC-16_3.9x9.9mm_P1.27mm
Connections:
- net MCU_SOL_0: now also R?.1, R?.1, U?.4 (I4); no longer R?.1, R?.1, U?.1 (I1)
- net MCU_SOL_1: now also R?.1, R?.1, U?.3 (I3); no longer R?.1, R?.1, U?.2 (I2)
- net MCU_SOL_2: now also R?.1, R?.1, U?.2 (I2); no longer R?.1, R?.1, U?.3 (I3)
- net MCU_SOL_3: now also R?.1, R?.1, U?.1 (I1); no longer R?.1, R?.1, U?.4 (I4)
- net MCU_SOL_4: now also R?.1, R?.1, U?.4 (I4); no longer R?.1, R?.1, U?.1 (I1)
- net MCU_SOL_5: now also R?.1, R?.1, U?.3 (I3); no longer R?.1, R?.1, U?.2 (I2)
- net MCU_SOL_6: now also R?.1, R?.1, U?.2 (I2); no longer R?.1, R?.1, U?.3 (I3)
- net MCU_SOL_7: now also R?.1, R?.1, U?.1 (I1); no longer R?.1, R?.1, U?.4 (I4)
- net MCU_SOL_8: now also R?.1, R?.1, U?.4 (I4); no longer R?.1, R?.1, U?.1 (I1)
- net MCU_SOL_9: now also R?.1, R?.1, U?.3 (I3); no longer R?.1, R?.1, U?.2 (I2)
- net MCU_SOL_A: now also R?.1, R?.1, U?.2 (I2); no longer R?.1, R?.1, U?.3 (I3)
- net MCU_SOL_B: now also R?.1, R?.1, U?.1 (I1); no longer R?.1, R?.1, U?.4 (I4)
- net MCU_SOL_C: now also R?.1, R?.1, U?.4 (I4); no longer R?.1, R?.1, U?.1 (I1)
- net MCU_SOL_D: now also R?.1, R?.1, U?.3 (I3); no longer R?.1, R?.1, U?.2 (I2)
- net MCU_SOL_E: now also R?.1, R?.1, U?.2 (I2); no longer R?.1, R?.1, U?.3 (I3)
- net MCU_SOL_F: now also R?.1, R?.1, U?.1 (I1); no longer R?.1, R?.1, U?.4 (I4)
- net SOL_0: now also U?.13 (O4); no longer U?.16 (O1)
- net SOL_1: now also U?.14 (O3); no longer U?.15 (O2)
- net SOL_2: now also U?.15 (O2); no longer U?.14 (O3)
- net SOL_3: now also U?.16 (O1); no longer U?.13 (O4)
- net SOL_4: now also U?.13 (O4); no longer U?.16 (O1)
- net SOL_5: now also U?.14 (O3); no longer U?.15 (O2)
- net SOL_6: now also U?.15 (O2); no longer U?.14 (O3)
- net SOL_7: now also U?.16 (O1); no longer U?.13 (O4)
- net SOL_8: now also U?.13 (O4); no longer U?.16 (O1)
- net SOL_9: now also U?.14 (O3); no longer U?.15 (O2)
- net SOL_A: now also U?.15 (O2); no longer U?.14 (O3)
- net SOL_B: now also U?.16 (O1); no longer U?.13 (O4)
- net SOL_C: now also U?.13 (O4); no longer U?.16 (O1)
- net SOL_D: now also U?.14 (O3); no longer U?.15 (O2)
- net SOL_E: now also U?.15 (O2); no longer U?.14 (O3)
- net SOL_F: now also U?.16 (O1); no longer U?.13 (O4)
- net at R?.1, R?.1, U?.6 (I6): no longer R?.1
- net at R?.1, U?.7 (I7): now also R?.1
- no-connect marks 0 -> 12

Commit message: finalize fab files and order first rev of board
Parts:
- J? (x2): now left out of the parts list
Changed lines of the file:
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@@
   )
   (symbol (lib_id "Connector_Generic:Conn_01x08") (at 52.705 178.435 0) (unit 1)
-    (in_bom yes) (on_board yes) (dnp no) (fields_autoplaced)
+    (in_bom no) (on_board yes) (dnp no) (fields_autoplaced)
     (property "Reference" "J?" (at 55.245 179.07 0)
       (effects (font (size 1.27 1.27)) (justify left))
@@
   )
   (symbol (lib_id "Connector_Generic:Conn_01x10") (at 95.885 175.895 0) (unit 1)
-    (in_bom yes) (on_board yes) (dnp no) (fields_autoplaced)
+    (in_bom no) (on_board yes) (dnp no) (fields_autoplaced)
     (property "Reference" "J?" (at 98.425 176.53 0)
       (effects (font (size 1.27 1.27)) (justify left))
